Commit message: Base hand movement finalised and Starting to run RL experiments

File: examples/allegro_hand_description/allegro_hand_description_left_digit.urdf (robot description, URDF)
Before this commit: robot allegro_hand_left, 21 links, 20 joints
Links:
- link base_link: mass None -> 30.0
Joints:
- joint joint_0.0: limit lower=-0.47 upper=0.47 effort=0 velocity=0 -> lower=-1.000 upper=1.000 effort=5.0 velocity=10.0
- joint joint_1.0: limit lower=-0.196 upper=1.61 effort=0 velocity=0 -> lower=-1.000 upper=1.000 effort=5.0 velocity=10.0
- joint joint_10.0: limit lower=-0.174 upper=1.709 effort=0 velocity=0 -> lower=-1.000 upper=1.000 effort=5.0 velocity=10.0
- joint joint_11.0: limit lower=-0.227 upper=1.618 effort=0 velocity=0 -> lower=-1.000 upper=1.000 effort=5.0 velocity=10.0
- joint joint_12.0: limit lower=0.263 upper=1.396 effort=0 velocity=0 -> lower=-1.000 upper=1.000 effort=5.0 velocity=10.0
- joint joint_13.0: limit lower=-0.105 upper=1.163 effort=0 velocity=0 -> lower=-1.000 upper=1.000 effort=5.0 velocity=10.0
- joint joint_14.0: limit lower=-0.189 upper=1.644 effort=0 velocity=0 -> lower=-1.000 upper=1.000 effort=5.0 velocity=10.0
- joint joint_15.0: limit lower=-0.162 upper=1.719 effort=0 velocity=0 -> lower=-1.000 upper=1.000 effort=5.0 velocity=10.0
- joint joint_2.0: limit lower=-0.174 upper=1.709 effort=0 velocity=0 -> lower=-1.000 upper=1.000 effort=5.0 velocity=10.0
- joint joint_3.0: limit lower=-0.227 upper=1.618 effort=0 velocity=0 -> lower=-1.000 upper=1.000 effort=5.0 velocity=10.0
- joint joint_4.0: limit lower=-0.47 upper=0.47 effort=0 velocity=0 -> lower=-1.000 upper=1.000 effort=5.0 velocity=10.0
- joint joint_5.0: limit lower=-0.196 upper=1.61 effort=0 velocity=0 -> lower=-1.000 upper=1.000 effort=5.0 velocity=10.0
- joint joint_6.0: limit lower=-0.174 upper=1.709 effort=0 velocity=0 -> lower=-1.000 upper=1.000 effort=5.0 velocity=10.0
- joint joint_7.0: limit lower=-0.227 upper=1.618 effort=0 velocity=0 -> lower=-1.000 upper=1.000 effort=5.0 velocity=10.0
- joint joint_8.0: limit lower=-0.47 upper=0.47 effort=0 velocity=0 -> lower=-1.000 upper=1.000 effort=5.0 velocity=10.0
- joint joint_9.0: limit lower=-0.196 upper=1.61 effort=0 velocity=0 -> lower=-1.000 upper=1.000 effort=5.0 velocity=10.0
