Commit message: StrixG16

File: examples/allegro_hand_description/allegro_hand_description_left_digit_fixed.urdf (robot description, URDF)
Before this commit: robot allegro_hand_left, 21 links, 20 joints
Links:
- link base_link: mass 30.0 -> 0.5
- link link_0.0: mass None -> 0.02
- link link_1.0: mass None -> 0.03
- link link_10.0: mass None -> 0.025
- link link_11.0: mass None -> 0.02
- link link_11.0_tip: mass None -> 0.01
- link link_12.0: mass None -> 0.035
- link link_13.0: mass None -> 0.02
- link link_14.0: mass None -> 0.025
- link link_15.0: mass None -> 0.02
- link link_15.0_tip: mass None -> 0.01
- link link_2.0: mass None -> 0.025
- link link_3.0: mass None -> 0.02
- link link_3.0_tip: mass None -> 0.01
- link link_4.0: mass None -> 0.02
- link link_5.0: mass None -> 0.03
- link link_6.0: mass None -> 0.025
- link link_7.0: mass None -> 0.02
- link link_7.0_tip: mass None -> 0.01
- link link_8.0: mass None -> 0.02
- link link_9.0: mass None -> 0.03
